File: KICAD/_autosave-MAX7000CPU-Gen2_5.sch (KiCad schematic (older format))
At the start: 72 parts

Commit message: A few changes to notes
Other:
- note removed: "Design Issues:\nNo Pulls on Register Reads\nNo Pulls on Instruction Expanders\nNo way to Set a constant (bypass buffer or something)"
